Commit message: 2021/6/2 commit

File: exoskeleton_description/urdf/lower_limb.urdf (robot description, URDF)
Before this commit: robot lower_limb, 10 links, 9 joints
Links:
- link Back_Base_Link: mass 7.1666344893724 -> 0.000000000001; geometry collision mesh filename=package://exoskeleton_description/meshes/Back_Base_Link.STL; visual mesh filename=package://exoskeleton_description/meshes/Back_Base_Link.STL
- link Left_Hip_Link: geometry collision mesh filename=package://exoskeleton_description/meshes/Left_Hip_Link.STL; visual mesh filename=package://exoskeleton_description/meshes/Left_Hip_Link.STL
